Commit message: Realizado el archivo URDF para el arduinobot

File: src/arduinobot_description/urdf/arduinobot.urdf.xacro (robot description, xacro)
@@ -1 +1,109 @@
 <?xml version="1.0"?>
+<robot xmlns:xacro="http://www.ros.org/wiki/xacro" name="arduinobot">
+    <xacro:property name="PI" value="3.14159"/>
+    <xacro:property name="effort" value="30.0"/>
+    <xacro:property name="velocity" value="10.0"/>
+    <link name="world"/>
+    <link name="base_link">
+        <visual>
+            <origin rpy="0 0 0" xyz="-0.5 -0.5 0"/>
+            <geometry>
+                <mesh filename="package://arduinobot_description/meshes/basement.stl" scale="0.01 0.01 0.01"/>
+            </geometry>
+        </visual>
+    </link>
+    <joint name="virtual_joint" type="fixed">
+        <parent link="world"/>
+        <child link="base_link"/>
+        <origin rpy="0 0 0" xyz="0 0 0"/>
+    </joint>
+    <link name="base_plate">
+        <visual>
+            <origin rpy="0 0 0" xyz="-0.39 -0.39 -0.56"/>
+            <geometry>
+                <mesh filename="package://arduinobot_description/meshes/base_plate.STL" scale="0.01 0.01 0.01"/>
+            </geometry>
+        </visual>
+    </link>
+    <joint name="joint_1" type="revolute">
+        <parent link="base_link"/>
+        <child link="base_plate"/>
+        <axis xyz="0.0 0.0 1.0"/>
+        <origin rpy="0 0 0" xyz="0 0 0.307"/>
+        <limit lower="-${PI/2}" upper="${PI/2}" effort="${effort}" velocity="${velocity}"/>
+    </joint>
+    <link name="forward_drive_arm">
+        <visual>
+            <origin rpy="0 -${PI/2} ${PI/2}" xyz="0.19 0.06 -0.08"/>
+            <geometry>
+                <mesh filename="package://arduinobot_description/meshes/forward_drive_arm.stl" scale="0.01 0.01 0.01"/>
+            </geometry>
+        </visual>
+    </link>
+    <joint name="joint_2" type="revolute">
+        <parent link="base_plate"/>
+        <child link="forward_drive_arm"/>
+        <axis xyz="1.0 0.0 0.0"/>
+        <origin rpy="0 0 0" xyz="-0.02 0 0.35"/>
+        <limit lower="-${PI/2}" upper="${PI/2}" effort="${effort}" velocity="${velocity}"/>
+    </joint>
+    <link name="horizontal_arm">
+        <visual>
+            <origin rpy="${PI/2} 0.0 ${PI/2}" xyz="-0.03 -0.4 -0.06"/>
+            <geometry>
+                <mesh filename="package://arduinobot_description/meshes/horizontal_arm.stl" scale="0.01 0.01 0.01"/>
+            </geometry>
+        </visual>
+    </link>
+    <joint name="joint_3" type="revolute">
+        <origin xyz="0.0 0.0 0.8" rpy="0.0 0.0 0.0"/>
+        <parent link="forward_drive_arm"/>
+        <child link="horizontal_arm"/>
+        <axis xyz="1.0 0.0 0.0"/>
+        <limit lower="-${PI/2}" upper="${PI/2}" effort="${effort}" velocity="${velocity}"/>
+    </joint>
+    <link name="claw_support">
+        <visual>
+            <origin xyz="0 -0.5 -0.15" rpy="0.0 0.0 ${PI/2}"/>
+            <geometry>
+                <mesh filename="package://arduinobot_description/meshes/claw_support.stl" scale="0.01 0.01 0.01"/>
+            </geometry>
+        </visual>
+    </link>
+<joint name="horizontal_arm_to_claw_support" type="fixed">
+    <origin xyz="0 0.82 0" rpy="0.0 0.0 0.0"/>
+    <parent link="horizontal_arm"/>
+    <child link="claw_support"/>
+</joint>
+<link name="gripper_right">
+    <visual>
+        <origin xyz="-0.1 0.5 -0.1" rpy="0.0 0.0 -${PI/2}"/>
+        <geometry>
+            <mesh filename="package://arduinobot_description/meshes/right_finger.stl" scale="0.01 0.01 0.01"/>
+        </geometry>
+    </visual>
+</link>
+<link name="gripper_left">
+    <visual>
+        <origin xyz="-0.04 0.5 -0.1" rpy="0.0 0.0 -${PI/2}"/>
+        <geometry>
+            <mesh filename="package://arduinobot_description/meshes/left_finger.stl" scale="0.01 0.01 0.01"/>
+        </geometry>
+    </visual>
+</link>
+<joint name="joint_4" type="revolute">
+    <origin xyz="-0.04 0.13 -0.1" rpy="0.0 0.0 0.0"/>
+    <parent link="claw_support"/>
+    <child link="gripper_right"/>
+    <axis xyz="0.0 0.0 1.0"/>
+    <limit lower="-${PI/2}" upper="0.0" effort="${effort}" velocity="${velocity}"/>
+</joint>
+<joint name="joint_5" type="revolute">
+    <origin xyz="-0.22 0.13 -0.1" rpy="0.0 0.0 0.0"/>
+    <parent link="claw_support"/>
+    <child link="gripper_left"/>
+    <axis xyz="0.0 0.0 1.0"/>
+    <limit lower="0.0" upper="${PI/2}" effort="${effort}" velocity="${velocity}"/>
+    <mimic joint="joint_4" multiplier="-1"/>
+</joint>
+</robot>

Commit message: Añadido matrices de inercia al URDF

File: src/arduinobot_description/urdf/arduinobot.urdf.xacro (robot description, xacro)
@@ -4,6 +4,15 @@
     <xacro:property name="effort" value="30.0"/>
     <xacro:property name="velocity" value="10.0"/>
+    <xacro:macro name="default_inertial" params="mass">
+        <inertial>
+                <mass value="${mass}"/>
+                <inertia    ixx="1" ixy="0.0" ixz="0.0"
+                            iyy="1" iyz="0.0"
+                            izz="1"/>
+        </inertial>
+    </xacro:macro>
     <link name="world"/>
     <link name="base_link">
+        <xacro:default_inertial mass="1.0"/>
         <visual>
             <origin rpy="0 0 0" xyz="-0.5 -0.5 0"/>
@@ -12,4 +21,10 @@
             </geometry>
         </visual>
+        <collision>
+            <origin rpy="0 0 0" xyz="-0.5 -0.5 0"/>
+            <geometry>
+                <mesh filename="package://arduinobot_description/meshes/basement.stl" scale="0.01 0.01 0.01"/>
+            </geometry>
+        </collision>
     </link>
     <joint name="virtual_joint" type="fixed">
@@ -19,4 +34,5 @@
     </joint>
     <link name="base_plate">
+        <xacro:default_inertial mass="0.1"/>
         <visual>
             <origin rpy="0 0 0" xyz="-0.39 -0.39 -0.56"/>
@@ -25,4 +41,10 @@
             </geometry>
         </visual>
+        <collision>
+            <origin rpy="0 0 0" xyz="-0.39 -0.39 -0.56"/>
+            <geometry>
+                <mesh filename="package://arduinobot_description/meshes/base_plate.STL" scale="0.01 0.01 0.01"/>
+            </geometry>
+        </collision>
     </link>
     <joint name="joint_1" type="revolute">
@@ -34,4 +56,5 @@
     </joint>
     <link name="forward_drive_arm">
+        <xacro:default_inertial mass="0.1"/>
         <visual>
             <origin rpy="0 -${PI/2} ${PI/2}" xyz="0.19 0.06 -0.08"/>
@@ -40,4 +63,10 @@
             </geometry>
         </visual>
+        <collision>
+            <origin rpy="0 -${PI/2} ${PI/2}" xyz="0.19 0.06 -0.08"/>
+            <geometry>
+                <mesh filename="package://arduinobot_description/meshes/forward_drive_arm.stl" scale="0.01 0.01 0.01"/>
+            </geometry>
+        </collision>
     </link>
     <joint name="joint_2" type="revolute">
@@ -49,4 +78,5 @@
     </joint>
     <link name="horizontal_arm">
+        <xacro:default_inertial mass="0.1"/>
         <visual>
             <origin rpy="${PI/2} 0.0 ${PI/2}" xyz="-0.03 -0.4 -0.06"/>
@@ -55,4 +85,10 @@
             </geometry>
         </visual>
+        <collision>
+            <origin rpy="${PI/2} 0.0 ${PI/2}" xyz="-0.03 -0.4 -0.06"/>
+            <geometry>
+                <mesh filename="package://arduinobot_description/meshes/horizontal_arm.stl" scale="0.01 0.01 0.01"/>
+            </geometry>
+        </collision>
     </link>
     <joint name="joint_3" type="revolute">
@@ -64,4 +100,5 @@
     </joint>
     <link name="claw_support">
+        <xacro:default_inertial mass="0.05"/>
         <visual>
             <origin xyz="0 -0.5 -0.15" rpy="0.0 0.0 ${PI/2}"/>
@@ -70,4 +107,10 @@
             </geometry>
         </visual>
+        <collision>
+            <origin xyz="0 -0.5 -0.15" rpy="0.0 0.0 ${PI/2}"/>
+            <geometry>
+                <mesh filename="package://arduinobot_description/meshes/claw_support.stl" scale="0.01 0.01 0.01"/>
+            </geometry>
+        </collision>
     </link>
     <joint name="horizontal_arm_to_claw_support" type="fixed">
@@ -77,4 +120,5 @@
     </joint>
     <link name="gripper_right">
+        <xacro:default_inertial mass="0.01"/>
         <visual>
             <origin xyz="-0.1 0.5 -0.1" rpy="0.0 0.0 -${PI/2}"/>
@@ -83,6 +127,13 @@
             </geometry>
         </visual>
+        <collision>
+            <origin xyz="-0.1 0.5 -0.1" rpy="0.0 0.0 -${PI/2}"/>
+            <geometry>
+                <mesh filename="package://arduinobot_description/meshes/right_finger.stl" scale="0.01 0.01 0.01"/>
+            </geometry>
+        </collision>
     </link>
     <link name="gripper_left">
+        <xacro:default_inertial mass="0.01"/>
         <visual>
             <origin xyz="-0.04 0.5 -0.1" rpy="0.0 0.0 -${PI/2}"/>
@@ -91,4 +142,10 @@
             </geometry>
         </visual>
+        <collision>
+            <origin xyz="-0.04 0.5 -0.1" rpy="0.0 0.0 -${PI/2}"/>
+            <geometry>
+                <mesh filename="package://arduinobot_description/meshes/left_finger.stl" scale="0.01 0.01 0.01"/>
+            </geometry>
+        </collision>
     </link>
     <joint name="joint_4" type="revolute">
@@ -114,4 +171,10 @@
             </geometry>
         </visual>
+        <collision>
+            <origin xyz="-0.05 0 0" rpy=" -1.57 0 -1.57"/>
+            <geometry>
+                <box size="0.30 0.30 0.10"/>
+            </geometry>
+            </collision>
     </link>
     <joint name="camera_fixed_joint" type="fixed">

Commit message: Sigue sin funcionar. Cambiado el gitignore para mayor comodidad

File: src/arduinobot_description/urdf/arduinobot.urdf.xacro (robot description, xacro)
@@ -1,4 +1,5 @@
 <?xml version="1.0"?>
 <robot xmlns:xacro="http://www.ros.org/wiki/xacro" name="arduinobot">
+    <xacro:arg name="is_ignition" default="false"/>
     <xacro:property name="PI" value="3.14159"/>
     <xacro:property name="effort" value="30.0"/>
@@ -165,4 +166,5 @@
     </joint>
     <link name="rgb_camera">
+        <xacro:default_inertial mass="0.001"/>
         <visual>
             <origin xyz="-0.09 0.125 0.135" rpy=" -1.57 0 -1.57"/>
@@ -176,5 +178,5 @@
                 <box size="0.30 0.30 0.10"/>
             </geometry>
-            </collision>
+        </collision>
     </link>
     <joint name="camera_fixed_joint" type="fixed">
@@ -183,3 +185,36 @@
         <child link="rgb_camera"/>
     </joint>
+ <gazebo reference="rgb_camera">
+    <sensor name="camera" type="camera">
+        <always_on>true</always_on>
+        <update_rate>30.0</update_rate>
+        <visualize>true</visualize>
+        <topic>/image_raw</topic>
+        <gz_frame_id>/rgb_camera</gz_frame_id>
+        <camera name="camera">
+          <horizontal_fov>1.21126</horizontal_fov>
+          <image>
+            <width>2304</width>
+            <height>1296</height>
+            <format>R8G8B8</format>
+          </image>
+          <distortion>
+            <k1>0.0</k1>
+            <k2>0.0</k2>
+            <k3>0.0</k3>
+            <p1>0.0</p1>
+            <p2>0.0</p2>
+            <center>0.5 0.5</center>
+          </distortion>
+        </camera>
+    </sensor>
+</gazebo>
+<gazebo>
+    <plugin filename="gz_ros2_control-system" name="gz_ros2_control::GazeboSimROS2ControlPlugin">
+      <parameters></parameters>
+    </plugin>
+    <plugin filename="gz-sim-sensors-system" name="gz::sim::systems::Sensors">
+      <render_engine>ogre2</render_engine>
+    </plugin>
+</gazebo>
 </robot>

Commit message: stl to STL para los meshes en ubuntu

File: src/arduinobot_description/urdf/arduinobot.urdf.xacro (robot description, xacro)
@@ -21,5 +21,5 @@
             <origin rpy="0 0 0" xyz="-0.5 -0.5 0"/>
             <geometry>
-                <mesh filename="package://arduinobot_description/meshes/basement.stl" scale="0.01 0.01 0.01"/>
+                <mesh filename="package://arduinobot_description/meshes/basement.STL" scale="0.01 0.01 0.01"/>
             </geometry>
         </visual>
@@ -27,5 +27,5 @@
             <origin rpy="0 0 0" xyz="-0.5 -0.5 0"/>
             <geometry>
-                <mesh filename="package://arduinobot_description/meshes/basement.stl" scale="0.01 0.01 0.01"/>
+                <mesh filename="package://arduinobot_description/meshes/basement.STL" scale="0.01 0.01 0.01"/>
             </geometry>
         </collision>
@@ -63,5 +63,5 @@
             <origin rpy="0 -${PI/2} ${PI/2}" xyz="0.19 0.06 -0.08"/>
             <geometry>
-                <mesh filename="package://arduinobot_description/meshes/forward_drive_arm.stl" scale="0.01 0.01 0.01"/>
+                <mesh filename="package://arduinobot_description/meshes/forward_drive_arm.STL" scale="0.01 0.01 0.01"/>
             </geometry>
         </visual>
@@ -69,5 +69,5 @@
             <origin rpy="0 -${PI/2} ${PI/2}" xyz="0.19 0.06 -0.08"/>
             <geometry>
-                <mesh filename="package://arduinobot_description/meshes/forward_drive_arm.stl" scale="0.01 0.01 0.01"/>
+                <mesh filename="package://arduinobot_description/meshes/forward_drive_arm.STL" scale="0.01 0.01 0.01"/>
             </geometry>
         </collision>
@@ -85,5 +85,5 @@
             <origin rpy="${PI/2} 0.0 ${PI/2}" xyz="-0.03 -0.4 -0.06"/>
             <geometry>
-                <mesh filename="package://arduinobot_description/meshes/horizontal_arm.stl" scale="0.01 0.01 0.01"/>
+                <mesh filename="package://arduinobot_description/meshes/horizontal_arm.STL" scale="0.01 0.01 0.01"/>
             </geometry>
         </visual>
@@ -91,5 +91,5 @@
             <origin rpy="${PI/2} 0.0 ${PI/2}" xyz="-0.03 -0.4 -0.06"/>
             <geometry>
-                <mesh filename="package://arduinobot_description/meshes/horizontal_arm.stl" scale="0.01 0.01 0.01"/>
+                <mesh filename="package://arduinobot_description/meshes/horizontal_arm.STL" scale="0.01 0.01 0.01"/>
             </geometry>
         </collision>
@@ -107,5 +107,5 @@
             <origin xyz="0 -0.5 -0.15" rpy="0.0 0.0 ${PI/2}"/>
             <geometry>
-                <mesh filename="package://arduinobot_description/meshes/claw_support.stl" scale="0.01 0.01 0.01"/>
+                <mesh filename="package://arduinobot_description/meshes/claw_support.STL" scale="0.01 0.01 0.01"/>
             </geometry>
         </visual>
@@ -113,5 +113,5 @@
             <origin xyz="0 -0.5 -0.15" rpy="0.0 0.0 ${PI/2}"/>
             <geometry>
-                <mesh filename="package://arduinobot_description/meshes/claw_support.stl" scale="0.01 0.01 0.01"/>
+                <mesh filename="package://arduinobot_description/meshes/claw_support.STL" scale="0.01 0.01 0.01"/>
             </geometry>
         </collision>
@@ -127,5 +127,5 @@
             <origin xyz="-0.1 0.5 -0.1" rpy="0.0 0.0 -${PI/2}"/>
             <geometry>
-                <mesh filename="package://arduinobot_description/meshes/right_finger.stl" scale="0.01 0.01 0.01"/>
+                <mesh filename="package://arduinobot_description/meshes/right_finger.STL" scale="0.01 0.01 0.01"/>
             </geometry>
         </visual>
@@ -133,5 +133,5 @@
             <origin xyz="-0.1 0.5 -0.1" rpy="0.0 0.0 -${PI/2}"/>
             <geometry>
-                <mesh filename="package://arduinobot_description/meshes/right_finger.stl" scale="0.01 0.01 0.01"/>
+                <mesh filename="package://arduinobot_description/meshes/right_finger.STL" scale="0.01 0.01 0.01"/>
             </geometry>
         </collision>
@@ -142,5 +142,5 @@
             <origin xyz="-0.04 0.5 -0.1" rpy="0.0 0.0 -${PI/2}"/>
             <geometry>
-                <mesh filename="package://arduinobot_description/meshes/left_finger.stl" scale="0.01 0.01 0.01"/>
+                <mesh filename="package://arduinobot_description/meshes/left_finger.STL" scale="0.01 0.01 0.01"/>
             </geometry>
         </visual>
@@ -148,5 +148,5 @@
             <origin xyz="-0.04 0.5 -0.1" rpy="0.0 0.0 -${PI/2}"/>
             <geometry>
-                <mesh filename="package://arduinobot_description/meshes/left_finger.stl" scale="0.01 0.01 0.01"/>
+                <mesh filename="package://arduinobot_description/meshes/left_finger.STL" scale="0.01 0.01 0.01"/>
             </geometry>
         </collision>
@@ -172,5 +172,5 @@
             <origin xyz="-0.09 0.125 0.135" rpy=" -1.57 0 -1.57"/>
             <geometry>
-                <mesh filename="package://arduinobot_description/meshes/pi_camera.stl" scale="0.01 0.01 0.01"/>
+                <mesh filename="package://arduinobot_description/meshes/pi_camera.STL" scale="0.01 0.01 0.01"/>
             </geometry>
         </visual>
